File: PWR_Supply/file5AB361F6.sch (KiCad schematic (older format))
At the start: 3 parts, among them U1 LM7805_TO220

Commit message: 1.1
Changed lines of the file:
@@
 LIBS:contrib
 LIBS:valves
+LIBS:PWR_Supply-cache
 EELAYER 25 0
 EELAYER END
@@
 Wire Wire Line
 	3400 2550 3400 2900
+$Comp
+L PWR_FLAG #FLG03
+U 1 1 5AB3AC59
+P 3650 2900
+F 0 "#FLG03" H 3650 2975 50  0001 C CNN
+F 1 "PWR_FLAG" H 3650 3050 50  0000 C CNN
+F 2 "" H 3650 2900 50  0001 C CNN
+F 3 "" H 3650 2900 50  0001 C CNN
+	1    3650 2900
+	-1   0    0    1
+$EndComp
+Wire Wire Line
+	3650 2900 3650 2850
+Wire Wire Line
+	3650 2850 3400 2850
+Connection ~ 3400 2850
 $EndSCHEMATC
