File: Шушурин(Susurina)_AMP/Шушурин(Susurina)_AMP.sch (KiCad schematic (older format))
At the start: 58 parts

Commit message: 5.0
Gala darbs
Connections:
- net GNDD: now also Output1.1 (Pin_1); no longer Output1.2 (Pin_2)
- net at C7.1, R16.1, R22.2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: now also Output1.2 (Pin_2); no longer Output1.1 (Pin_1)
Changed lines of the file:
@@
 L Conn_01x02 Output1
 U 1 1 5AF69FF7
-P 7700 3250
-F 0 "Output1" H 7700 3350 50  0000 C CNN
-F 1 "Conn_01x02" H 7700 3050 50  0000 C CNN
-F 2 "Connectors_Terminal_Blocks:TerminalBlock_Altech_AK300-2_P5.00mm" H 7700 3250 50  0001 C CNN
-F 3 "" H 7700 3250 50  0001 C CNN
-	1    7700 3250
-	1    0    0    -1
+P 7700 3350
+F 0 "Output1" H 7700 3450 50  0000 C CNN
+F 1 "Conn_01x02" H 7700 3150 50  0000 C CNN
+F 2 "Connectors_Terminal_Blocks:TerminalBlock_Altech_AK300-2_P5.00mm" H 7700 3350 50  0001 C CNN
+F 3 "" H 7700 3350 50  0001 C CNN
+	1    7700 3350
+	1    0    0    1
 $EndComp
 $Comp
